File: upd78214-breakout.kicad_pcb (KiCad board)
At the start: 2 copper layers, 1 part, among them U1 upd78214-64p-qfp

Commit message: Add attempt at PCB
Routing:
- net unconnected-(U1-Pad28): track 0.00 -> 14.5 mm
- net unconnected-(U1-Pad54): track 0.00 -> 13.6 mm
- net unconnected-(U1-Pad26): track 0.00 -> 13.6 mm
- net unconnected-(U1-Pad55): track 0.00 -> 12.8 mm
- net unconnected-(U1-Pad25): track 0.00 -> 12.2 mm
- net unconnected-(U1-Pad56): track 0.00 -> 12.1 mm
- net unconnected-(U1-Pad24): track 0.00 -> 11.5 mm
- net unconnected-(U1-Pad57): track 0.00 -> 11.4 mm
- net unconnected-(U1-Pad17): track 0.00 -> 11.3 mm
- net unconnected-(U1-Pad41): track 0.00 -> 11.2 mm
- net unconnected-(U1-Pad64): track 0.00 -> 11.2 mm
- net unconnected-(U1-Pad61): track 0.00 -> 11.2 mm
- net unconnected-(U1-Pad6): track 0.00 -> 11.1 mm
- net unconnected-(U1-Pad9): track 0.00 -> 11.0 mm
- net unconnected-(U1-Pad1): track 0.00 -> 10.9 mm
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Other:
- board text added: "10"
- board text added: "11"
- board text added: "12"
- board text added: "12.5V GND"
- board text added: "12.5V PS"
- board text added: "13"
- board text added: "2"
- board text added: "20"
- board text added: "21"
- board text added: "22"
- board text added: "24"
- board text added: "25"
- board text added: "26"
- board text added: "27"
- board text added: "28"
- board text added: "3"
- board text added: "30"
- board text added: "31"
- board text added: "32"
- board text added: "33"
- board text added: "34"
- board text added: "35"
- board text added: "36"
- board text added: "37"
- board text added: "4"
- board text added: "5"
- board text added: "6"
- board text added: "7"
- board text added: "8"
- board text added: "9"
- board text added: "Mega GND"
