File: upd78214-arduino-mega-hat/upd78214-arduino-mega-hat.kicad_pcb (KiCad board)
At the start: 4 copper layers, 101.6 x 53.3 mm, 20 parts, among them J1 Power, J2 PWM, J3 Analog, J4 PWM, J5 Analog, J6 Communication, J7 Digital, J8 NMI +12V / GND, U1 upd78214-64p-qfp, Y1 4-12MHz

Commit message: More correct wiring for shield
Parts:
- added JP3: SolderJumper-2, Jumper:SolderJumper-2_P1.3mm_Bridged2Bar_RoundedPad1.0x1.5mm, F.Cu at (115.5, 86.0)
- added R1: 10k, Capacitor_SMD:C_0805_2012Metric_Pad1.18x1.45mm_HandSolder, F.Cu at (114.0, 76.5)
- added R10: 10k, Capacitor_SMD:C_0805_2012Metric_Pad1.18x1.45mm_HandSolder, F.Cu at (134.3, 73.0)
- added R11: 10k, Capacitor_SMD:C_0805_2012Metric_Pad1.18x1.45mm_HandSolder, F.Cu at (158.3, 64.7)
- added R12: 10k, Capacitor_SMD:C_0805_2012Metric_Pad1.18x1.45mm_HandSolder, F.Cu at (158.0, 61.2)
- added R13: 10k, Capacitor_SMD:C_0805_2012Metric_Pad1.18x1.45mm_HandSolder, F.Cu at (162.4, 60.5)
- added R14: 10k, Capacitor_SMD:C_0805_2012Metric_Pad1.18x1.45mm_HandSolder, F.Cu at (158.5, 59.1)
- added R15: 10k, Capacitor_SMD:C_0805_2012Metric_Pad1.18x1.45mm_HandSolder, F.Cu at (157.9, 57.3)
- added R16: 10k, Capacitor_SMD:C_0805_2012Metric_Pad1.18x1.45mm_HandSolder, F.Cu at (134.0, 58.2)
- added R17: 10k, Capacitor_SMD:C_0805_2012Metric_Pad1.18x1.45mm_HandSolder, F.Cu at (112.5, 72.6)
- added R18: 10k, Capacitor_SMD:C_0805_2012Metric_Pad1.18x1.45mm_HandSolder, F.Cu at (146.8, 58.3)
- added R19: 10k, Capacitor_SMD:C_0805_2012Metric_Pad1.18x1.45mm_HandSolder, F.Cu at (112.5, 84.9)
- added R2: 10k, Capacitor_SMD:C_0805_2012Metric_Pad1.18x1.45mm_HandSolder, F.Cu at (114.0, 78.6)
- added R20: 10k, Capacitor_SMD:C_0805_2012Metric_Pad1.18x1.45mm_HandSolder, F.Cu at (170.0, 60.5)
- added R3: 10k, Capacitor_SMD:C_0805_2012Metric_Pad1.18x1.45mm_HandSolder, F.Cu at (114.0, 80.7)
- added R4: 10k, Capacitor_SMD:C_0805_2012Metric_Pad1.18x1.45mm_HandSolder, F.Cu at (114.0, 82.8)
- added R5: 10k, Capacitor_SMD:C_0805_2012Metric_Pad1.18x1.45mm_HandSolder, F.Cu at (108.0, 61.1)
- added R6: 10k, Capacitor_SMD:C_0805_2012Metric_Pad1.18x1.45mm_HandSolder, F.Cu at (108.0, 63.2)
- added R7: 10k, Capacitor_SMD:C_0805_2012Metric_Pad1.18x1.45mm_HandSolder, F.Cu at (169.5, 75.6)
- added R8: 10k, Capacitor_SMD:C_0805_2012Metric_Pad1.18x1.45mm_HandSolder, F.Cu at (109.5, 74.7)
- added R9: 10k, Capacitor_SMD:C_0805_2012Metric_Pad1.18x1.45mm_HandSolder, F.Cu at (162.4, 66.6)
Connections:
- J2 pad 2: /SDA/20 -> /a3
- J2 pad 6: /*12 -> /a7
- J2 pad 7: /*11 -> /a6
- J2 pad 8: /*10 -> /a5
- J2 pad 9: /*9 -> /a4
- J4 pad 4: /*4 -> /a2
- J4 pad 5: /*3 -> /a1
- J4 pad 6: /*2 -> /a0
- J6 pad 1: /TX3/14 -> /prog_a9
- J7 pad 27: /28 -> /upd_oe
- J7 pad 29: /26 -> /upd_ea
- J7 pad 30: /27 -> /upd_ce
- J7 pad 31: /24 -> /upd_reset
- U1 pad 1: unconnected-(U1-p6,4/~{RD}-Pad1) -> /upd_oe
- U1 pad 2: unconnected-(U1-p6,3/a19-Pad2) -> /pd02
- U1 pad 29: unconnected-(U1-p2,1/intp0-Pad29) -> /prog_a9
- U1 pad 3: unconnected-(U1-p6,2/a18-Pad3) -> /pd03
- U1 pad 30: unconnected-(U1-p2,2/intp1-Pad30) -> GND
- U1 pad 31: unconnected-(U1-p2,3/intp2/ci-Pad31) -> GND
- U1 pad 32: unconnected-(U1-p2,4/intp3-Pad32) -> GND
- U1 pad 33: unconnected-(U1-p2,5/intp4/asck-Pad33) -> GND
- U1 pad 34: unconnected-(U1-p2,6/intp5-Pad34) -> GND
- U1 pad 35: unconnected-(U1-p2,7/si-Pad35) -> GND
- U1 pad 38: unconnected-(U1-p3,2/sck-Pad38) -> /pd38
- U1 pad 39: unconnected-(U1-p3,3/so/sb0-Pad39) -> /pd39
- U1 pad 4: unconnected-(U1-p6,1/a17-Pad4) -> /pd04
- U1 pad 40: unconnected-(U1-~{EA}-Pad40) -> /upd_ea
- U1 pad 43: +5V -> /pd43
- U1 pad 44: unconnected-(U1-p7,5/AN5-Pad44) -> /pd44
- U1 pad 45: unconnected-(U1-p7,4/AN4-Pad45) -> /pd45
- U1 pad 46: unconnected-(U1-p7,3/AN3-Pad46) -> /pd46
- U1 pad 47: unconnected-(U1-p7,2/AN2-Pad47) -> /pd47
- U1 pad 48: unconnected-(U1-p7,1/AN1-Pad48) -> /pd48
- U1 pad 49: unconnected-(U1-p7,0/AN0-Pad49) -> /pd49
- U1 pad 5: unconnected-(U1-p6,0/a16-Pad5) -> /pd05
- U1 pad 54: unconnected-(U1-p0,0-Pad54) -> /a0
- U1 pad 55: unconnected-(U1-p0,1-Pad55) -> /a1
- U1 pad 56: unconnected-(U1-p0,2-Pad56) -> /a2
- U1 pad 57: unconnected-(U1-p0,3-Pad57) -> /a3
- U1 pad 58: unconnected-(U1-p0,4-Pad58) -> /a4
- U1 pad 59: unconnected-(U1-p0,5-Pad59) -> /a5
- U1 pad 6: unconnected-(U1-~{RESET}-Pad6) -> /upd_reset
- U1 pad 60: unconnected-(U1-p0,6-Pad60) -> /a6
- U1 pad 61: unconnected-(U1-p0,7-Pad61) -> /a7
- U1 pad 62: unconnected-(U1-p6,7/~{REFRQ}/AN7-Pad62) -> /pd62
- U1 pad 63: unconnected-(U1-p6,6/~{WAIT}/AN6-Pad63) -> /pd63
- U1 pad 64: unconnected-(U1-p6,5/~{WR}-Pad64) -> /upd_ce
Routing:
- net /upd_reset: track 0.00 -> 169.6 mm, vias 0 -> 2
- net /upd_ce: track 0.00 -> 150.3 mm, vias 0 -> 5
- net /upd_oe: track 0.00 -> 108.0 mm
- net /prog_a9: track 0.00 -> 98.7 mm
- net /a4: track 0.00 -> 71.6 mm
- net /upd_ea: track 0.00 -> 69.1 mm, vias 0 -> 3
- net GND: track 9.79 -> 77.0 mm, vias 6 -> 18
- net /a5: track 0.00 -> 64.4 mm
- net /a3: track 0.00 -> 63.7 mm, vias 0 -> 2
- net /a6: track 0.00 -> 56.2 mm
- net /pd38: track 0.00 -> 51.1 mm, vias 0 -> 1
- net /a0: track 0.00 -> 49.2 mm, vias 0 -> 1
- net /a7: track 0.00 -> 49.0 mm
- net /a1: track 0.00 -> 48.0 mm
- net /a2: track 0.00 -> 46.8 mm, vias 0 -> 1
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