File: upd78214-arduino-mega-hat/upd78214-arduino-mega-hat.kicad_sch (KiCad schematic)
At the start: 18 parts, among them J1 Power, J2 PWM, J3 Analog, J4 PWM, J5 Analog, J6 Communication, J7 Digital, J8 Conn_01x02, SW1 SW_SPST, SW2 SW_SPDT, U1 upd78214-64p-qfp, Y1 4-12MHz

Commit message: More correct wiring for shield
Parts:
- added JP3: Jumper_2_Bridged, Jumper:SolderJumper-2_P1.3mm_Bridged2Bar_RoundedPad1.0x1.5mm, symbol Jumper:Jumper_2_Bridged
- added R10, R11, R12, R13, R14, R15, R16, R17, R18, R19, R20, R3, R4, R5, R6, R7, R8, R9: 10kΩ, Capacitor_SMD:C_0805_2012Metric_Pad1.18x1.45mm_HandSolder, symbol Device:R_Small_US
- R1, R2: footprint (none) -> Capacitor_SMD:C_0805_2012Metric_Pad1.18x1.45mm_HandSolder
Connections:
- net 23 is gone; now on an unnamed net: J7.34 (Pin_34)
- net ~{RESET} is gone; now on net +5V: J1.3 (Pin_3)
- net +5V: now also R17.2, R18.1, R19.2, R20.1; no longer J1.5 (Pin_5), J7.35 (Pin_35), J7.36 (Pin_36), U1.41 (Vdd)
- net GND: now also C1.1, J1.1 (Pin_1), U1.42 (AVss), JP3.2 (B), R10.2, R11.1, R12.1, R13.1, R14.1, R15.1, R16.1, R3.2, R4.2, R5.2, R6.2, R7.1, R8.2, R9.1; no longer C1.2, J1.6 (Pin_6), J1.7 (Pin_7), J2.4 (Pin_4), J7.1 (Pin_1), J7.2 (Pin_2)
- net VCC: no longer J1.8 (Pin_8)
- net at SW1.1 (A): no longer U1.7 (X2)
- net Net-(U1-X2): now reaches C2.1, Y1.2
- net Net-(U1-X2): now also JP3.1 (A); no longer SW1.2 (B)
- net at U1.43 (AVref): no longer R1.1
- net /pd03: now reaches R2.1
- net /pd03: no longer U1.42 (AVss)
- net at SW2.2 (B): no longer U1.8 (X1)
- net Net-(JP1-B): now reaches JP1.2 (B), U1.37 (p3,1/txd)
- net Net-(JP2-B): now reaches JP2.2 (B), U1.36 (p3,0/rxd)
- net *10: no longer names the net of J2.8 (Pin_8)
- net *11: no longer names the net of J2.7 (Pin_7)
- net *12: no longer names the net of J2.6 (Pin_6)
- net *13: no longer names the net of J2.5 (Pin_5)
- net *2: no longer names the net of J4.6 (Pin_6)
- net *3: no longer names the net of J4.5 (Pin_5)
- net *4: no longer names the net of J4.4 (Pin_4)
- net *5: no longer names the net of J4.3 (Pin_3)
- net *6: no longer names the net of J4.2 (Pin_2)
- net *7: no longer names the net of J4.1 (Pin_1)
- net *9: no longer names the net of J2.9 (Pin_9)
- net 22: no longer names the net of J7.33 (Pin_33)
- net 24 renamed /ad7
- net 25 renamed /a15
- net 26 renamed /ad6
- net 27 renamed /a14
- net 28 renamed /ad5
- net 29 renamed /a13
- net 30 renamed /ad4
- net 31 renamed /a12
- net 32 renamed /ad3
- net 33 renamed /a11
- net 34 renamed /ad2
- net 35 renamed /a10
- net 36 renamed /ad1
- net 37 renamed /a9
- net /a9: now also R7.2
- net A0 renamed /A6
- net A1 renamed /A5
- net A10 renamed /A12
- net A11 renamed /A11
- net A12 renamed /A10
- net A13 renamed /A9
- net A14 renamed /A8
- net A15: no longer names the net of J5.8 (Pin_8)
- net A2 renamed /A4
- net A3 renamed /A3
- net A4 renamed /A2
- net A5 renamed /A1
- net A6 renamed /A0
- net A7: no longer names the net of J3.8 (Pin_8)
- net A8 renamed /A14
- net A9 renamed /A13
- net AREF: no longer names the net of J2.3 (Pin_3)
- net IOREF: no longer names the net of J1.2 (Pin_2)
- net RX0/0: no longer names the net of J4.8 (Pin_8)
- net RX0/0: no longer JP1.1 (A)
- net RX1/19: no longer names the net of J6.6 (Pin_6)
- net RX2/17: no longer names the net of J6.4 (Pin_4)
- net RX3/15: no longer names the net of J6.2 (Pin_2)
- net SCL/21: no longer names the net of J2.1 (Pin_1)
- net SCL/21: no longer J6.8 (Pin_8)
- net SDA/20: no longer names the net of J2.2 (Pin_2)
- net SDA/20: no longer J6.7 (Pin_7)
- net TX0/1: no longer names the net of J4.7 (Pin_7)
- net TX0/1: no longer JP2.1 (A)
- net TX1/18: no longer names the net of J6.5 (Pin_5)
- net TX2/16: no longer names the net of J6.3 (Pin_3)
- net TX3/14: no longer names the net of J6.1 (Pin_1)
- net a10: no longer names the net of U1.15 (p5,2/a10)
- net a10: no longer J7.14 (Pin_14)
- net a11: no longer names the net of U1.14 (p5,3/a11)
- net a11: no longer J7.12 (Pin_12)
- net a12: no longer names the net of U1.13 (p5,4/a12)
- net a12: no longer J7.10 (Pin_10)
- net a13: no longer names the net of U1.12 (p5,5/a13)
- net a13: no longer J7.8 (Pin_8)
- net a14: no longer names the net of U1.11 (p5,6/a14)
- net a14: no longer J7.6 (Pin_6)
- net a15: no longer names the net of U1.10 (p5,7/a15)
- net a15: no longer J7.4 (Pin_4)
- net a8: no longer names the net of U1.17 (p5,0/a8)
- net a8: no longer J7.18 (Pin_18)
- net a9: no longer names the net of U1.16 (p5,1/a9)
- net a9: no longer J7.16 (Pin_16)
- net ad0: no longer names the net of U1.26 (p4,0/ad0)
- net ad0: no longer J7.17 (Pin_17)
- net ad1: no longer names the net of U1.25 (p4,1/ad1)
- net ad1: no longer J7.15 (Pin_15)
- net ad2: no longer names the net of U1.23 (p4,2/ad2)
- net ad2: no longer J7.13 (Pin_13)
- net ad3: no longer names the net of U1.22 (p4,3/ad3)
- net ad3: no longer J7.11 (Pin_11)
- net ad4: no longer names the net of U1.21 (p4,4/ad4)
- net ad4: no longer J7.9 (Pin_9)
- net ad5: no longer names the net of U1.20 (p4,5/ad5)
- net ad5: no longer J7.7 (Pin_7)
- net ad6: no longer names the net of U1.19 (p4,6/ad6)
- net ad6: no longer J7.5 (Pin_5)
- net ad7: no longer names the net of U1.18 (p4,7/ad7)
- net ad7: no longer J7.3 (Pin_3)
- new net /22: J7.1 (Pin_1)
- new net /23: J7.2 (Pin_2)
- new net /25: J7.4 (Pin_4)
- new net /29: J7.8 (Pin_8)
- new net /30: J7.9 (Pin_9)
- new net /31: J7.10 (Pin_10)
- new net /32: J7.11 (Pin_11)
- new net /33: J7.12 (Pin_12)
- new net /34: J7.13 (Pin_13)
- new net /35: J7.14 (Pin_14)
- new net /36: J7.15 (Pin_15)
- new net /37: J7.16 (Pin_16)
- new net /IOREF: J1.6 (Pin_6)
- new net /RX0/0: JP1.1 (A)
- new net /TX0/1: JP2.1 (A)
- new net /a8: J7.18 (Pin_18)
- new net /ad0: J7.17 (Pin_17)
- new net /pd02: R1.1
- new net /pd04: R3.1
- new net /pd05: R4.1
- new net /pd38: R8.1
- new net /pd39: R9.2
- new net /pd43: R10.1
- new net /pd44: R11.2
- new net /pd45: R12.2
- new net /pd46: R13.2
- new net /pd47: R14.2
- new net /pd48: R15.2
- new net /pd49: R16.2
- new net /pd62: R5.1
- new net /pd63: R6.1
- new net /upd_ce: J7.6 (Pin_6), R18.2
- new net /upd_ea: J7.5 (Pin_5), R20.2
- new net /upd_oe: J7.7 (Pin_7), R17.1
- new net /upd_reset: J7.3 (Pin_3), R19.1
- new net /~{RESET}: J1.5 (Pin_5)
- new net Net-(U1-X1): C1.2, Y1.1
- now unconnected: SW2.1 (A)
